File: Ligther/Ligther.kicad_sch (KiCad schematic)
At the start: 42 parts, among them Q1 IRF9622, Q2 IRFZ24N, Q3 BC547, Q4 IRF9622, SW1 SW_Reed, U1 NE555P, U2 BCR421U

Commit message: Add pcb and production files
Parts:
- removed JP13, JP14: Jumper_2_Open, symbol Jumper:Jumper_2_Open
- removed Q4: IRF9622, Package_TO_SOT_THT:TO-220-3_Vertical, symbol Transistor_FET:IRF4905
- removed R10: 100R, Resistor_THT:R_Axial_DIN0207_L6.3mm_D2.5mm_P10.16mm_Horizontal, symbol Device:R
- added R17: 4K, Resistor_THT:R_Axial_DIN0207_L6.3mm_D2.5mm_P10.16mm_Horizontal, symbol Device:R
- JP1, JP10, JP11, JP12, JP2, JP3, JP4, JP5, JP6, JP7, JP8, JP9: footprint (none) -> Connector_PinHeader_1.27mm:PinHeader_2x01_P1.27mm_Vertical
- R6: value 2.4K -> 3K
Connections:
- net +4.5V is gone; now on net +6V: SW1.1
- net +6V_Safe is gone; now on net +6VS: Q1.3 (S), R2.1, U1.4 (R), U1.8 (VCC)
- net +6V: no longer R5.2
- net GND: no longer U2.4 (GND)
- net GNDPWR: now also U2.4 (GND), R17.1; no longer Q3.3 (E)
- net +6VS: now reaches D1.4 (A), D2.4 (A), D3.4 (A), R6.2
- net +6VS: now also R5.2
- net LED_C: now reaches D1.2 (R), D2.2 (R), D3.2 (R), U2.2 (OUT), U2.3 (OUT), U2.5 (OUT)
- new net: Q3.3 (E), R17.2
